Commit message: Added lidar detection and changed wheel color to purple

File: description/robot.urdf.xacro (robot description, xacro)
@@ -3,3 +3,5 @@
     <!-- Example link -->
    <xacro:include filename="robot_core.xacro" />
+   <xacro:include filename="gazebo_control.xacro"/>
+   <xacro:include filename="lidar.xacro"/>
 </robot>

File: description/robot_core.xacro (robot description, xacro)
@@ -5,4 +5,7 @@
      <material name="white">
         <color rgba="1 1 1 1"/>
+     </material>
+     <material name="purple">
+         <color rgba="0.607 0.043 0.871 1"/>
      </material>
      <material name = "orange">
@@ -44,4 +47,9 @@
          </xacro:inertial_box>
      </link>
+   <gazebo reference ="chassis">
+      <material>
+         Gazebo/White
+      </material>
+   </gazebo>
      <!-- Left Drive Wheel-->
      <joint name="LW_joint" type="continuous">
@@ -56,5 +64,5 @@
                <cylinder radius="0.05" length="0.04"/>
             </geometry>
-            <material name="black"/>
+            <material name="purple"/>
          </visual>
          <collision>
@@ -67,4 +75,9 @@
          </xacro:inertial_cylinder>
       </link>
+      <gazebo reference ="left_wheel">
+         <material>
+            Gazebo/Purple
+         </material>
+      </gazebo>
       <!-- Right Drive Wheel-->
      <joint name="RW_joint" type="continuous">
@@ -79,5 +92,5 @@
                <cylinder radius="0.05" length="0.04"/>
             </geometry>
-            <material name="black"/>
+            <material name="purple"/>
          </visual>
          <collision>
@@ -90,4 +103,9 @@
          </xacro:inertial_cylinder>
       </link>
+      <gazebo reference ="right_wheel">
+         <material>
+            Gazebo/Purple
+         </material>
+      </gazebo>
       <!-- Caster Wheel-->
        <joint name="CW_joint" type="fixed">
@@ -101,5 +119,5 @@
                <sphere radius="0.05"/>
             </geometry>
-               <material name="blue"></material>
+               <material name="black"></material>
          </visual>
          <collision>
@@ -112,3 +130,10 @@
          </xacro:inertial_sphere>
        </link>
+       <gazebo reference ="caster_wheel">
+         <material>
+            Gazebo/Black
+         </material>
+         <mu1 value="0.001"/>
+         <mu2 value="0.001"/>
+      </gazebo>
 </robot>
