Commit message: SLAM Added using cartogropher+New world

File: description/lidar.xacro (robot description, xacro)
@@ -4,5 +4,5 @@
             <parent link="chassis"/>
             <child link="laser_frame"/>
-            <origin xyz="0.1 0 0.175" rpy="0 0 0"/>
+            <origin xyz="0.24 0 0.175" rpy="0 0 0"/>
         </joint>
         <link name="laser_frame">
@@ -18,5 +18,5 @@
                 </geometry>
             </collision>
-            <xacro:inertial_cylinder mass="0.1" length="0.04" radius="0.05">
+            <xacro:inertial_cylinder mass="0.5" length="0.04" radius="0.05">
                 <origin xyz="0 0 0" rpy="0 0 0"/>
             </xacro:inertial_cylinder>
@@ -24,5 +24,5 @@
     <gazebo reference="laser_frame">
         <sensor name="laser" type="ray">
-            <pose>0 0 0 0 0 0</pose>
+            <pose>0.24 0 0.175 0 0 0</pose>
             <visualize>true</visualize>
             <update_rate>10</update_rate>
@@ -38,4 +38,5 @@
                 <range>
                     <min>0.3</min>
+                    <!--<max>12</max>-->
                     <max>12</max>
                     <resolution>0.01</resolution>

File: description/robot.urdf.xacro (robot description, xacro)
@@ -1,4 +1,4 @@
 <?xml version="1.0"?>
-<robot xmlns:xacro="http://www.ros.org/wiki/xacro"  name="robot">
+<robot xmlns:xacro="http://www.ros.org/wiki/xacro"  name="talos">
     <!-- Example link -->
    <xacro:include filename="robot_core.xacro" />
