Commit message: Fixed robot going all the way up issue
Co-authored-by: Copilot <copilot@github.com>

File: description/gazebo_control.xacro (robot description, xacro)
@@ -20,3 +20,10 @@
     </plugin>
    </gazebo>
+   <!-- Joint State Publisher for caster wheel -->
+   <gazebo>
+    <plugin name="joint_state_publisher" filename="libgazebo_ros_joint_state_publisher.so">
+        <joint_name>CW_joint</joint_name>
+        <update_rate>30</update_rate>
+    </plugin>
+   </gazebo>
 </robot>

File: description/robot_core.xacro (robot description, xacro)
@@ -109,5 +109,5 @@
       </gazebo>
       <!-- Caster Wheel-->
-       <joint name="CW_joint" type="fixed">
+       <joint name="CW_joint" type="continuous">
          <parent link="chassis"/>
          <child link="caster_wheel"/>
